File: ds8.sch (EAGLE design)
At the start: 93 parts, among them IC1 TM4C1230C3PM, IC2 TPS77333, Q1 BC850, Q2 BC850, Q3 BC850, U1 LM13700M, U2 LM324, U3 LM324, U4 LM741D, X1 MAB5SH

Commit message: Board retouted
- Cleaned the schematic
- Board rerouted with through hole pots and new connectors
- Lots of little stuff

Signed-off-by: Kamel Makhloufi <melka@blaste.net>
Parts:
- removed CV_IN, OUT: 3.5 JACK, SparkFun-Connectors:M03PTH
- removed MODE: 50K LOG, SparkFun-Connectors:M03PTH
- removed OK1: 6N138, optocoupler:6N138
- removed PAN: 50K LIN, SparkFun-Connectors:M03PTH
- removed POWER: 9V, SparkFun-Connectors:M02PTH
- removed RATE: 2M LIN, SparkFun-Connectors:M03PTH
- removed SC: ROCKER_SWITCH, SparkFun-Connectors:M03PTH
- added J1: 9VDC, SparkFun-Connectors:POWER_JACKPTH_LOCK
- added JP1: (no value), SparkFun-Connectors:AUDIO-JACK2.5MM
- added LFO_MODE: 50k LOG, SparkFun-Electromechanical:POTALPS-KIT
- added LFO_RATE: 2M LIN, SparkFun-Electromechanical:POTALPS-KIT
- added NOISE_MIX: 50k LIN, SparkFun-Electromechanical:POTALPS-KIT
- added U$3: ALPS_SRBV, ds8:ALPS_SRBV
- added U$4: OPTO_DARL_6N138S, SparkFun-DiscreteSemi:OPTO_DARL_6N138S
- D3: value 1N4148DO35-7 -> 4148; device diode:1N4148DO35-7 -> diode:DIODE-MINIMELF
- DECAY: value 500K LIN -> 500k LIN; device SparkFun-Connectors:M03PTH -> SparkFun-Electromechanical:POTALPS-KIT
- LEVEL, SWEEP, VCO: value 50K LOG -> 50k LOG; device SparkFun-Connectors:M03PTH -> SparkFun-Electromechanical:POTALPS-KIT
- TRIGGER: value 3.5 JACK -> M02PTH; device SparkFun-Connectors:M03PTH -> SparkFun-Connectors:M02PTH
Connections:
- net N$34 renamed TRIGGER
- removed net PAN1: PAN.1, R20.2, R33.2
- removed net PAN2: PAN.2
- removed net PAN3: PAN.3, R101.2, R34.1
- removed net SC1: C10.2, SC.1
- removed net SC2: C5.2, R35.2, SC.2, U4.-IN
- removed net SC3: C11.2, SC.3
- removed net TRIG: RV1.CCW, TRIGGER.2, TRIGGER.3
- removed net VCO1: R11.2, VCO.1
- removed net VCO3: R10.2, VCO.3
- new net N$34: RV1.CCW, TRIGGER.2
- new net N$37: R10.2, VCO.E
- new net N$38: R11.2, VCO.A
- new net N$39: C10.1, U$3.P$3
- new net N$40: C11.1, U$3.P$1
- new net NOISECOLOR_2: C5.2, R35.2, U$3.P$2, U4.-IN
- new net NOISEMIX_1: NOISE_MIX.A, R20.2, R33.2
- new net NOISEMIX_3: NOISE_MIX.E, R101.2, R34.1
- net /RESET: now also R40.1; no longer R40.2
- net 9VDC: now also J1.PWR; no longer POWER.1
- net CVIN: no longer CV_IN.2, CV_IN.3
- net DECAY: now also DECAY.E; no longer DECAY.3
- net GND: now also C10.2, C11.2, C15.2, DECAY.A, DECAY.S, J1.GND, J1.GNDBREAK, JP1.SLEEVE, LEVEL.A, LFO_MODE.A, NOISE_MIX.S, SWEEP.A, U$4.GND; no longer C10.1, C11.1, C15.1, CV_IN.1, DECAY.1, DECAY.2, LEVEL.1, MODE.1, OK1.GND, OUT.1, POWER.2, SWEEP.1
- net LFO2: now also LFO_MODE.S; no longer MODE.2
- net LFO3: now also LFO_MODE.E; no longer MODE.3
- net MIDI_IN: now also U$4.VOUT; no longer OK1.VO
- net N$26: now also U$4.A; no longer OK1.A
- net N$28: now also U4.OUT
- net N$35: now also U$4.C; no longer OK1.C
- net N$36: now also C15.1; no longer C15.2
- net N$5: now also R5.1
- net N$57: now also JP1.LEFT, JP1.RIGHT, LEVEL.S; no longer LEVEL.2, OUT.2, OUT.3
- net OUT: now also LEVEL.E; no longer LEVEL.3
- net S2: now also LFO_RATE.E; no longer RATE.3
- net S3: now also LFO_RATE.A, LFO_RATE.S; no longer RATE.1, RATE.2
- net SWEEP2: now also SWEEP.S; no longer SWEEP.2
- net SWEEP3: now also SWEEP.E; no longer SWEEP.3
- net VCC: now also U$4.VCC; no longer OK1.VCC
- net VCO2: now also VCO.S; no longer VCO.2
- net VDD: now also R40.2; no longer R40.1
Other:
- note added: "5V -> 3.3V"
- note added: "9V -> 5V"
- note added: "ANALOG"
- note added: "CONTROLS"
- note added: "ENVELOPE"
- note added: "LOGIC"
- note added: "NOISE"
- note added: "OUTPUT"
- note added: "PIEZO"
- note added: "POWER SUPPLY"
- note added: "UNUSED"
- note removed: "Controls"
- note removed: "Envelope"
- note removed: "Noise"
- note removed: "Output"
- note removed: "Power Supply"
- moved on the sheet: C1, C10, C100, C101, C11, C12, C13, C14, C15, C2, C3, C4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
